File: pcb/65C816.kicad_pcb (KiCad board)
At the start: 2 copper layers, 100 x 41.4 mm, 13 parts, among them J1 Conn_02x05_Odd_Even, J2 Conn_02x06_Odd_Even, J3 Conn_02x06_Odd_Even, J4 Conn_02x06_Odd_Even, J5 Conn_02x06_Odd_Even, U1 65C816S, U2 AS6C4008

Commit message: Upgrade Kicad projects to v6
Connections:
- net /R~W renamed /R~{W}
- net /~ABORT renamed /~{ABORT}
- net /~CE renamed /~{CE}
- net /~IRQ renamed /~{IRQ}
- net /~ML renamed /~{ML}
- net /~NMI renamed /~{NMI}
- net /~OE renamed /~{OE}
- net /~RES renamed /~{RES}
- net /~VP renamed /~{VP}
- net /~WE renamed /~{WE}
Other:
- net class Default removed
